File: project/BGKiCad.kicad_pcb (KiCad board)
At the start: 2 copper layers, 50.8 x 50.8 mm, 1 part

Commit message: Add reversible hotswap Choc footprint
Parts:
- added SW1: SW_choc_v1_HS_CPG135001S30_1u_Reversible, BGKiCad:SW_choc_v1_HS_CPG135001S30_1u_Reversible, F.Cu at (62.9, 39.4)
Connections:
- D1 pad 2: unconnected-(D1-A-Pad2) -> GND
Routing:
- added copper zone on B.Cu, net GND
- added copper zone on F.Cu, net GND
Other:
- board size 50.8 x 50.8 mm -> 63.5 x 50.8 mm
